File: Hardware/ReflowESP.sch (KiCad schematic (older format))
At the start: 58 parts, among them J1 USB_B_Micro, J2 SSR1, J3 SSR2, J4 SSR3, J5 TC1, J6 TC2, Q1 BSS138, Q2 BSS138, Q3 S8050, Q4 S8050, Q5 BSS138, SW1 SW_RESET, SW2 SW_BOOT, U1 CH340G, U2 NCP1117-3.3_SOT223, U3 ESP32-WROOM-32D, U4 MAX31855KASA, U5 MAX31855KASA, Y1 12MHz

Commit message: Update for v0.0.2
Migrate to KiCad 6
Switch to WROVER-E module and update symbol
Mechanical components
Parts:
- added D?: 1N5819, Diode_THT:D_DO-41_SOD81_P10.16mm_Horizontal, symbol Diode:1N5819
- gave numbers to parts that had none: 2
- renumbered J1 to J2, J2 to J3, J3 to J5, J4 to J6, J5 to J7, J6 to J8, JP4 to JP1
Connections:
- net at J1.4 (Pin_4): now also D?.1 (K); no longer J1.2 (Pin_2)
- new net: D?.2 (A), J1.2 (Pin_2)
Other:
- note added: "Two jumpers are used\nto set the desired V_SSR.\n3v3, 5v, or an external source."
- note removed: "TODO: Rework this.\nAlso, maybe add diodes to prevent\nsending EXT_V_SSR to 5V line."
- moved on the sheet: J4
