File: Hardware/ReflowESP.kicad_sch (KiCad schematic)
At the start: 58 parts, among them J1 USB_B_Micro, J10 SSR3, J11 TC1, J12 TC2, J2 VIN, J3 PROG, J4 SERVO, J5 DISPLAY, J6 V_SSR_SEL, J7 SSR1, J8 EXT_V_SSR, J9 SSR2, Q1 BSS138, Q2 BSS138, Q3 BSS138, SW1 SW_RESET, SW2 SW_BOOT, U1 NCP1117-3.3_SOT223, U2 ESP32-WROVER-E, U3 MAX31855KASA, U4 MAX31855KASA

Commit message: Mostly finished layout
Parts:
- removed C2: 10u, symbol Device:C_Polarized
- removed J3: PROG, Connector_PinHeader_2.54mm:PinHeader_1x05_P2.54mm_Vertical, symbol Connector:Conn_01x05_Male
- added C2: 10u, Capacitor_SMD:C_0805_2012Metric, symbol Device:C
- added J3: PROG, Connector_PinHeader_2.54mm:PinHeader_1x06_P2.54mm_Vertical, symbol Connector:Conn_01x06_Male
- added R11: 220, Resistor_SMD:R_0805_2012Metric, symbol Device:R
- added TP1, TP2: TestPoint, TestPoint:TestPoint_Pad_D1.0mm, symbol Connector:TestPoint
- C3: footprint (none) -> Capacitor_SMD:CP_Elec_4x5.4
- J1: footprint (none) -> Connector_USB:USB_Micro-B_Molex_47346-0001
- J10, J11, J12, J2, J7, J8, J9: footprint (none) -> TerminalBlock_KF301:TerminalBlock_KF301-2P
- JP1: footprint Jumper:SolderJumper-2_P1.3mm_Bridged2Bar_RoundedPad1.0x1.5mm -> Jumper:SolderJumper-2_P1.3mm_Bridged_RoundedPad1.0x1.5mm
- L1, L2, L3, L4: footprint (none) -> Inductor_SMD:L_0805_2012Metric
- LS1: footprint (none) -> Buzzer_Beeper:MagneticBuzzer_ProSignal_ABI-010-RC
- SW1, SW2: footprint (none) -> Button_Switch_SMD:SW_Push_SPST_NO_Alps_SKRK
- renumbered R11 to R12, R12 to R13
Connections:
- net +3V3: now also J3.4 (Pin_4), TP2.1
- net +5V: now also C2.1, TP1.1
- net BUZZER: now also R11.1; no longer JP1.1 (A)
- net EN: now also J3.5 (Pin_5)
- net GND: now also C2.2, J3.1 (Pin_1)
- net IO0: now also J3.6 (Pin_6)
- net RX: now also J3.3 (Pin_3)
- net TX: now also J3.2 (Pin_2)
- new net: JP1.1 (A), R11.2
Other:
- note removed: "MLCC or tantalum"
- company: Doofenshmirtz Evil Inc -> Thomas Aldrian

Commit message: Update schematic symbols for connectors
Parts:
- removed J3: PROG, Connector_PinHeader_2.54mm:PinHeader_1x06_P2.54mm_Vertical, symbol Connector:Conn_01x06_Male
- removed J4: SERVO, Connector_PinHeader_2.54mm:PinHeader_1x03_P2.54mm_Horizontal, symbol Connector:Conn_01x03_Male
- added J3: PROG, Connector_PinHeader_2.54mm:PinHeader_1x06_P2.54mm_Vertical, symbol Connector_Generic:Conn_01x06
- added J4: SERVO, Connector_PinHeader_2.54mm:PinHeader_1x03_P2.54mm_Horizontal, symbol Connector_Generic:Conn_01x03
- J5: symbol Connector:Conn_01x07_Male -> Connector_Generic:Conn_01x07
Connections:
- net +3V3: now also J3.3 (Pin_3)
- net +5V: now also J4.2 (Pin_2)
- net EN: now also J3.2 (Pin_2)
- net GND: now also J3.6 (Pin_6), J4.1 (Pin_1)
- net IO0: now also J3.1 (Pin_1)
- net PWM: now also J4.3 (Pin_3)
- net RX: now also J3.4 (Pin_4)
- net TX: now also J3.5 (Pin_5)
