File: Hardware/ReflowESP.kicad_sch (KiCad schematic)
At the start: 61 parts, among them J1 USB_B_Micro, J10 SSR3, J11 TC1, J12 TC2, J2 VIN, J3 PROG, J4 SERVO, J5 DISPLAY, J6 V_SSR_SEL, J7 SSR1, J8 EXT_V_SSR, J9 SSR2, Q1 BSS138, Q2 BSS138, Q3 BSS138, SW1 SW_RESET, SW2 SW_BOOT, U1 NCP1117-3.3_SOT223, U2 ESP32-WROVER-E, U3 MAX31855KASA, U4 MAX31855KASA

Commit message: Update v0.0.7
Add rotary encoder
Parts:
- added J7: Conn_01x05, Connector_PinHeader_2.54mm:PinHeader_1x05_P2.54mm_Vertical, symbol Connector_Generic:Conn_01x05
- added R7, R9: 10k, Resistor_SMD:R_0805_2012Metric, symbol Device:R_Small
- D1: footprint Diode_SMD:D_SOD-323 -> Diode_SMD:D_SOD-123
- renumbered C5 to C1, C6 to C11, C13 to C12, C11 to C13, C7 to C2, C12 to C3, C8 to C4, C9 to C5, C1 to C6, C2 to C7, C3 to C8, C4 to C9, H3 to H2, H2 to H3, J2 to J1, J6 to J10, J7 to J11, J9 to J12, J10 to J13, J1 to J2, J11 to J3, J3 to J5, J5 to J6, J12 to J8, J8 to J9, R2 to R1, R5 to R10, R7 to R11, R9 to R12, R6 to R13, R8 to R14, R10 to R15, R11 to R2, R1 to R3, R3 to R4, R4 to R5, R12 to R6, R13 to R8, U3 to U2, U2 to U3
Connections:
- net +3V3: now also J7.1 (Pin_1), R7.1, R9.1
- net GND: now also J7.5 (Pin_5)
- net RE_A: now reaches U3.6 (GPIO34/ADC1_CH6)
- net RE_A: now also J7.2 (Pin_2), R9.2
- net RE_B: now reaches U3.7 (GPIO35/ADC1_CH7)
- net RE_B: now also J7.3 (Pin_3), R7.2
- net MOSI renamed RE_SW
- net RE_SW: now also J7.4 (Pin_4)
- no-connect marks 9 -> 7
