File: Hardware/ReflowESP.kicad_pcb (KiCad board)
At the start: 2 copper layers, 72 x 72 mm, 61 parts, among them J1 USB_B_Micro, J10 SSR3, J11 TC1, J12 TC2, J2 VIN, J3 PROG, J4 SERVO, J5 DISPLAY, J6 V_SSR_SEL, J7 SSR1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

Commit message: Update PCB
Add pin 1 marker for U3 and U4
Add pinout for J4 and J5 to back silkscreen
Remove hole part designators
Parts:
- U3, U4: footprint Package_SO:SOIC-8_3.9x4.9mm_P1.27mm -> Package_SOIC-8:SOIC-8_3.9x4.9mm_P1.27mm
- moved J3 12.7 mm to (58.4, 38.1), turned to -90 degrees
Connections:
- J3 pad 1: GND -> IO0
- J3 pad 2: TX -> EN
- J3 pad 3: RX -> +3V3
- J3 pad 4: +3V3 -> RX
- J3 pad 5: EN -> TX
- J3 pad 6: IO0 -> GND
Routing:
- net V_CS0: track 33.8 -> 34.6 mm
- net GND: vias 127 -> 114
